Commit message: Added custom node to link ros2 cmd_vel with gazebo joints. Simulating movement in gazebo

File: cestra_description/urdf/diff_drive/diff_wheels.urdf.xacro (robot description, xacro)
@@ -17,5 +17,5 @@
     <collision>
         <geometry>
-            <sphere radius="${diff_wheel_radius}"/>
+            <cylinder length="${diff_wheel_width}" radius="${diff_wheel_radius}" />
         </geometry>
     </collision>

Commit message: Adding odom to wheels

File: cestra_description/urdf/diff_drive/diff_wheels.urdf.xacro (robot description, xacro)
@@ -4,5 +4,5 @@
     <joint name="${prefix}_wheel_joint" type="continuous">
         <parent link="base_link"/>
-        <child link="${prefix}_wheel"/>
+        <child  link="${prefix}_wheel"/>
         <origin xyz="0 ${diff_wheel_y * reflect} 0" rpy="${-pi/2 * reflect} 0 0"/>
         <axis xyz="0 0 ${reflect}"/>

Commit message: Added custom jsp and odom node

File: cestra_description/urdf/diff_drive/diff_wheels.urdf.xacro (robot description, xacro)
@@ -1,7 +1,7 @@
 <?xml version="1.0"?>
 <robot xmlns:xacro="http://www.ros.org/wiki/xacro" >
-<xacro:macro name="wheel" params="prefix reflect">
+<xacro:macro name="diff_wheel" params="prefix reflect">
     <joint name="${prefix}_wheel_joint" type="continuous">
-        <parent link="base_link"/>
+        <parent link="chassis"/>
         <child  link="${prefix}_wheel"/>
         <origin xyz="0 ${diff_wheel_y * reflect} 0" rpy="${-pi/2 * reflect} 0 0"/>
