Commit message: Fully functional swerve module for 4 wheels

File: cestra_description/urdf/cestra_swerve.urdf (robot description, URDF)
Before this commit: robot cestra_swerve, 4 links, 3 joints
Links:
- removed link steer_link
- removed link wheel_link
Joints:
- removed joint steer_joint
- removed joint wheel_joint
