Commit message: stuff

File: cestra_description/urdf/cestra_diff.urdf (robot description, URDF)
Before this commit: robot cestra, 3 links, 2 joints
Links:
- removed link chassis
- added link left_wheel, mass 0.1; collision cylinder length=0.02 radius=0.05; visual cylinder length=0.02 radius=0.05
- added link right_wheel, mass 0.1; collision cylinder length=0.02 radius=0.05; visual cylinder length=0.02 radius=0.05
- link base_link: mass None -> 0.5; geometry collision box size=0.30 0.30 0.15; visual box size=0.30 0.30 0.15
- link caster_wheel: mass None -> 0.05; geometry collision sphere radius=0.05; visual sphere radius=0.05
Joints:
- removed joint chassis_joint
- added joint left_wheel_joint: type continuous, parent base_link, child left_wheel, origin xyz=0 0.175 0 rpy=0 0 0, axis 0 1 0
- added joint right_wheel_joint: type continuous, parent base_link, child right_wheel, origin xyz=0 -0.175 0 rpy=0 0 0, axis 0 1 0
- joint caster_wheel_joint: origin xyz=0.24 0 0 rpy=0 0 0 -> xyz=0.10 0 0 rpy=0 0 0; parent chassis -> base_link

File: cestra_description/urdf/diff_drive/diff_wheels.urdf.xacro (robot description, xacro)
@@ -1,27 +1,36 @@
 <?xml version="1.0"?>
-<robot xmlns:xacro="http://www.ros.org/wiki/xacro" >
-<xacro:macro name="diff_wheel" params="prefix reflect">
+<robot xmlns:xacro="http://www.ros.org/wiki/xacro">
+  <xacro:macro name="diff_wheel"
+               params="prefix parent_link x y z roll pitch yaw">
     <joint name="${prefix}_wheel_joint" type="continuous">
-        <parent link="chassis"/>
-        <child  link="${prefix}_wheel"/>
-        <origin xyz="0 ${diff_wheel_y * reflect} 0" rpy="${-pi/2 * reflect} 0 0"/>
-        <axis xyz="0 0 ${reflect}"/>
+      <parent link="${parent_link}"/>
+      <child link="${prefix}_wheel"/>
+      <origin xyz="${x} ${y} ${z}"
+              rpy="${roll} ${pitch} ${yaw}"/>
+      <axis xyz="0 1 0"/>
     </joint>
     <link name="${prefix}_wheel">
-    <visual>
+      <visual>
+        <origin xyz="0 0 0" rpy="${pi/2} 0 0"/>
         <geometry>
-            <cylinder length="${diff_wheel_width}" radius="${diff_wheel_radius}" />
+          <cylinder radius="${diff_wheel_radius}"
+                    length="${diff_wheel_width}"/>
         </geometry>
         <material name="blue"/>
-    </visual>
-    <collision>
+      </visual>
+      <collision>
+        <origin xyz="0 0 0" rpy="${pi/2} 0 0"/>
         <geometry>
-            <cylinder length="${diff_wheel_width}" radius="${diff_wheel_radius}" />
+          <cylinder radius="${diff_wheel_radius}"
+                    length="${diff_wheel_width}"/>
         </geometry>
-    </collision>
-    <xacro:inertial_cylinder mass="0.1" length="0.05" radius="0.05">
-        <origin xyz="0 0 0" rpy="0 0 0"/>
-    </xacro:inertial_cylinder>
+      </collision>
+      <xacro:inertial_cylinder
+          mass="0.1"
+          length="${diff_wheel_width}"
+          radius="${diff_wheel_radius}">
+        <origin xyz="0 0 0" rpy="${pi/2} 0 0"/>
+      </xacro:inertial_cylinder>
     </link>
-</xacro:macro>
+  </xacro:macro>
 </robot>
